Commit message: Enhance haptic DMP learning and testing framework

File: src/testing_plane/xacro/testing_plane.xacro (robot description, xacro)
@@ -1,12 +1,28 @@
 <?xml version="1.0"?>
+<!--
+  6-DOF Testing Plane Model for Contact & Teleoperation Interaction in Gazebo Sim.
+  Kinematic Chain:
+    dummy_fixed_link (world anchor)
+      -> fixed_joint -> dummy_link
+      -> trasl_x_joint (prismatic X) -> trasl_x_link
+      -> trasl_y_joint (prismatic Y) -> trasl_y_link
+      -> trasl_z_joint (prismatic Z) -> trasl_z_link
+      -> rot_x_joint (revolute roll) -> rot_x_link
+      -> rot_y_joint (revolute pitch) -> rot_y_link
+      -> rot_z_joint (revolute yaw) -> rot_z_link
+      -> testing_plane_joint (fixed) -> testing_plane_link (physical red box)
+-->
 <robot xmlns:xacro="http://www.ros.org/wiki/xacro" name="testing_plane">
     <xacro:property name="robot_namespace" value="testing_plane"/>
-	<xacro:property name="h_testing_plane" value="0.1" />
-	<xacro:property name="l_testing_plane" value="0.1" />
-	<xacro:property name="w_testing_plane" value="0.1" />
+    <!-- Physical Box Dimensions (meters) -->
+    <xacro:property name="h_testing_plane" value="0.1" />
+    <xacro:property name="l_testing_plane" value="0.1" />
+    <xacro:property name="w_testing_plane" value="0.1" />
     <xacro:property name="absolute_height" value="1.0" />
+    <!-- Initial Position in Gazebo World -->
     <xacro:property name="initial_x" value="0.5" />
     <xacro:property name="initial_y" value="0.0" />
     <xacro:property name="initial_z" value="0.05" />
+    <!-- World Anchor Link -->
     <link name="${robot_namespace}_dummy_fixed_link">
          <inertial>
@@ -17,6 +33,6 @@
                 iyy="1e6" iyz="0.0"
                 izz="1e6"/>
-+        </inertial>
-+    </link>
+        </inertial>
+    </link>
     <joint name="${robot_namespace}_fixed_joint" type="fixed">
         <parent link="${robot_namespace}_dummy_fixed_link"/>

Commit message: Add free_target_object package and grasp_monitoring node
- Introduced a new package `free_target_object` which includes:
  - A model for a single free-floating rigid body in Gazebo, replacing the `testing_plane`.
  - Launch file to spawn the object in an existing Gazebo simulation.
  - Xacro file for model parameters including mass, size, and inertia.
  - CMake and package configuration files.

- Added `grasp_monitoring` package with a node to monitor geometric grasp:
  - Subscribes to the odometry of the target object and the end-effector pose via tf.
  - Emits a boolean signal indicating whether the grasp conditions are met based on position and alignment.
  - Includes parameters for tuning the grasp detection thresholds.

- Updated `testing_plane.launch.py` to use `ParameterValue` for URDF generation.
- Increased mass in `testing_plane.xacro` for simulation realism.

File: src/testing_plane/xacro/testing_plane.xacro (robot description, xacro)
@@ -236,5 +236,5 @@
     <link name="${robot_namespace}_link">
         <inertial>
-            <mass value="1.0" />
+            <mass value="5.0" />
             <origin xyz="0 0 0" rpy="0 0 0"/>
             <inertia
